File: Browse/rcbus-ymf262.kicad_pcb (KiCad board)
At the start: 2 copper layers, 100 x 50 mm, 42 parts, among them CON1 SJ1-3523N, P1 RC2014 BUS, U1 74HCT688, U2 YMF262, U3 YAC512, U4 TL074, X1 14.318MHz

Commit message: Deploying to main from @ electrified/rcbus-ymf262@09dfc0b6299e9abfa74e5c9ae499f817effffc48 🚀
Parts:
- removed X1: 14.318MHz, electrified:Oscillator_DIP-8-14
- added C19: 0.1uF, Capacitor_SMD:C_0603_1608Metric_Pad1.08x0.95mm_HandSolder, F.Cu at (101.2, 142.2)
- added Y1: SG-8002CA, Oscillator:Oscillator_SMD_Abracon_ASV-4Pin_7.0x5.1mm, F.Cu at (103.0, 146.8)
- moved G2 7.00 mm to (93.0, 128.0)
- moved C7 1.30 mm to (111.2, 143.0)
- moved C1 1.25 mm to (111.2, 156.8)
Routing:
- net /CLK: track 32.8 -> 10.9 mm
- net GND: track 79.5 -> 69.0 mm, vias 18 -> 17
- net /~{CS}: track 48.7 -> 51.7 mm
- net VCC: track 101.6 -> 98.9 mm, vias 1 -> 2
- net /D3: track 22.6 -> 23.6 mm
- net +5VA: track 57.3 -> 56.5 mm
- net /A7: track 7.13 -> 6.57 mm

Commit message: Deploying to main from @ electrified/rcbus-ymf262@b43f424ddd5021915e267e75a2a8900653243e1b 🚀
Parts:
- moved C6 0.66 mm to (80.0, 145.0), turned to 180 degrees
Routing:
- net VCC: track 98.9 -> 101.7 mm
- net GND: vias 17 -> 67

Commit message: Deploying to main from @ electrified/rcbus-ymf262@ffcfb9396d06d84fb116886ae824cff65907a9a5 🚀
Other:
- board text added: "Rev: ${VERSION} ${GIT_HASH}"
- board text removed: "Rev: @version@"

Commit message: Deploying to main from @ electrified/rcbus-ymf262@291c25c960d7e0f6c5c821497c85d57fa4939298 🚀
Parts:
- turned R1 to 0 degrees
- turned R2 to 0 degrees
- turned R3 to 0 degrees
- turned R4 to 0 degrees
- turned R5 to 0 degrees
- turned R6 to 0 degrees
Routing:
- net GND: track 69.0 -> 76.5 mm, vias 67 -> 73
- net VCC: track 101.7 -> 103.5 mm
- net Net-(JP1-Pin_1): track 30.2 -> 28.7 mm, vias 3 -> 2
- net Net-(JP1-Pin_3): track 32.3 -> 30.8 mm, vias 3 -> 2
- net Net-(JP1-Pin_7): track 29.5 -> 28.1 mm, vias 1 -> 0
- net Net-(JP1-Pin_5): track 30.9 -> 29.4 mm, vias 3 -> 2
- net Net-(JP1-Pin_11): track 35.8 -> 34.5 mm, vias 3 -> 2
- net Net-(JP1-Pin_9): track 30.0 -> 29.9 mm, vias 3 -> 2
