File: Browse/rcbus-ymf262.kicad_sch (KiCad schematic)
At the start: 40 parts, among them CON1 SJ1-3523N, P1 RC2014 BUS, U1 74HCT688, U2 YMF262, U3 YAC512, U4 TL074, X1 14.318MHz

Commit message: Deploying to main from @ electrified/rcbus-ymf262@09dfc0b6299e9abfa74e5c9ae499f817effffc48 🚀
Parts:
- removed X1: 14.318MHz, electrified:Oscillator_DIP-8-14, symbol electrified:CXO_DIP-8-14
- added C19: 0.1uF, Capacitor_SMD:C_0603_1608Metric_Pad1.08x0.95mm_HandSolder, symbol Device:C_Small
- added Y1: SG-8002CA, Oscillator:Oscillator_SMD_Abracon_ASV-4Pin_7.0x5.1mm, symbol Oscillator:ASV-xxxMHz
Connections:
- net CLK: now also Y1.3 (OUT)
- net GND: now also C19.2, Y1.2 (GND)
- net VCC: now also C19.1, Y1.1 (EN), Y1.4 (Vdd)
- no-connect marks 22 -> 21

Commit message: Deploying to main from @ electrified/rcbus-ymf262@b43f424ddd5021915e267e75a2a8900653243e1b 🚀
Parts:
- C8: symbol Device:C_Small -> Device:C_Polarized_Small
Changed lines of the file:
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@@
     )
   )
-  (symbol (lib_id "Device:C_Small") (at 262.89 80.01 0) (unit 1)
+  (symbol (lib_id "Device:C_Polarized_Small") (at 262.89 80.01 0) (unit 1)
     (exclude_from_sim no) (in_bom yes) (on_board yes) (dnp no)
     (property "Reference" "C8" (at 265.1252 78.8416 0)

Commit message: Deploying to main from @ electrified/rcbus-ymf262@9c8d0cd003b39a240463bae4e94c496cca633260 🚀
Connections:
- net AUDIO_CH1: now also C9.1, U4.10 (+); no longer C10.1, U4.12 (+)
- net AUDIO_CH2: now also C10.1, U4.12 (+); no longer C9.1, U4.10 (+)
- net L: now also C14.2, R9.2, U4.14; no longer C13.1, R8.2, U4.8
- net R: now also C13.1, R8.2, U4.8; no longer C14.2, R9.2, U4.14
Other:
- moved on the sheet: C10, C13, C14, C9, R8, R9, U4C, U4D
