File: Browse/rcbus-opl3.kicad_sch (KiCad schematic)
At the start: 37 parts, among them CON1 SJ1-3523N, P1 RC2014 BUS, U1 74HCT688, U2 YMF262, U3 YAC512, U4 TL074, Y1 SG-8002CA

Commit message: Deploying to main from @ electrified/rcbus-opl3@ca335f471b0cc053c0f7ada637c7f1deac17d0b8 🚀
Parts:
- removed C2: 10nF, Capacitor_SMD:C_0603_1608Metric, symbol Device:C_Small
- removed C3: 100nF, Capacitor_SMD:C_0603_1608Metric, symbol Device:C_Small
- removed C4: 10uF, Capacitor_SMD:C_1206_3216Metric, symbol Device:C_Polarized_Small
- removed L1: BLM18PG221SN1D, Inductor_SMD:L_0603_1608Metric, symbol Device:L
- removed L2: 33uH, Inductor_SMD:L_0603_1608Metric, symbol Device:L
- C15, C16: footprint Capacitor_SMD:CP_Elec_5x5.9 -> Capacitor_SMD:CP_Elec_6.3x5.8
- C5: value 10uF -> 100uF; footprint Capacitor_SMD:C_1206_3216Metric -> Capacitor_SMD:CP_Elec_6.3x7.7
- C8: footprint Capacitor_SMD:C_0603_1608Metric -> Capacitor_SMD:CP_Elec_6.3x5.8
Connections:
- net VCC is gone; now on net +5V: C1.1, C19.1, C6.1, JP1.10 (Pin_10), JP1.12 (Pin_12), JP1.2 (Pin_2), JP1.4 (Pin_4), JP1.6 (Pin_6), JP1.8 (Pin_8), P1.18 (Pin_18), U1.20 (VCC), U2.1 (VDD), Y1.1 (EN), Y1.4 (Vdd)
- net +5VA renamed +5V
Other:
- note added: "Line out"
- moved on the sheet: C1, C10, C11, C12, C15, C16, C19, C5, C6, C7, C8, C9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

Commit message: Deploying to main from @ electrified/rcbus-opl3@95905a1b3d61b904a2086439a003ecc01cce0db1 🚀
Parts:
- added C2: 10uf, Capacitor_SMD:CP_Elec_6.3x5.8, symbol Device:C_Polarized_Small
- CON1: value SJ1-3523N -> 3.5mm jack
- Y1: value SG-8002CA -> 14.3181MHz
Connections:
- net +5V: now also C2.1
- net GND: now also C2.2
Other:
- moved on the sheet: C5

Commit message: Deploying to main from @ electrified/rcbus-opl3@76df5429c526e7a9126e9bdce83f90b253efb9f7 🚀
Parts:
- C10: renamed from C2; value 10uf -> 10uF
- C3: renamed from C9; value 2.7nf -> 2.7nF
- C4: renamed from C10; value 2.7nf -> 2.7nF
- C5: renamed from C11; value 68pf -> 68pF
- C6: renamed from C16; value 10uf -> 10uF
- C7: renamed from C15; value 10uf -> 10uF
- renumbered C8 to C1, C6 to C11, C7 to C12, C19 to C13, C12 to C2, C1 to C8, C5 to C9, R7 to R1, R3 to R10, R6 to R11, R8 to R2, R9 to R3, R10 to R4, R11 to R5, R5 to R6, R4 to R7, R2 to R8, R1 to R9, U3 to U1, U4 to U2, U1 to U3, U2 to U4

Commit message: Deploying to main from @ electrified/rcbus-opl3@4d18163650932ad5441b7bd8b3289f36741a7241 🚀
Parts:
- renumbered C6 to C2, C4 to C3, C3 to C4, C2 to C5, C5 to C6, R4 to R2, R2 to R3, R3 to R4, R7 to R6, R6 to R7, U2 to U1, U1 to U2
Other:
- moved on the sheet: H1

Commit message: Deploying to main from @ electrified/rcbus-opl3@44c55904765375cbeefdfa411b2ca464d51f40a2 🚀
Other:
- moved on the sheet: C10, C9
Changed lines of the file:
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@@
   (junction (at 255.27 43.18) (diameter 0) (color 0 0 0 0)
   )
-  (junction (at 270.51 111.76) (diameter 0) (color 0 0 0 0)
+  (junction (at 87.63 59.69) (diameter 0) (color 0 0 0 0)
+  )
+  (junction (at 69.85 69.85) (diameter 0) (color 0 0 0 0)
+  )
+  (junction (at 44.45 59.69) (diameter 0) (color 0 0 0 0)
+  )
+  (junction (at 233.68 29.21) (diameter 0) (color 0 0 0 0)
+  )
+  (junction (at 69.85 67.31) (diameter 0) (color 0 0 0 0)
+  )
+  (junction (at 243.84 58.42) (diameter 0) (color 0 0 0 0)
+  )
+  (junction (at 50.8 67.31) (diameter 0) (color 0 0 0 0)
+  )
+  (junction (at 139.7 22.86) (diameter 0) (color 0 0 0 0)
+  )
+  (junction (at 237.49 109.22) (diameter 0) (color 0 0 0 0)
+  )
+  (junction (at 107.95 82.55) (diameter 0) (color 0 0 0 0)
+  )
+  (junction (at 69.85 64.77) (diameter 0) (color 0 0 0 0)
+  )
+  (junction (at 44.45 67.31) (diameter 0) (color 0 0 0 0)
+  )
+  (junction (at 82.55 149.86) (diameter 0) (color 0 0 0 0)
+  )
+  (junction (at 100.33 82.55) (diameter 0) (color 0 0 0 0)
+  )
+  (junction (at 50.8 77.47) (diameter 0) (color 0 0 0 0)
+  )
+  (junction (at 232.41 144.78) (diameter 0) (color 0 0 0 0)
+  )
+  (junction (at 195.58 97.79) (diameter 0) (color 0 0 0 0)
+  )
+  (junction (at 82.55 160.02) (diameter 0) (color 0 0 0 0)
+  )
+  (junction (at 237.49 82.55) (diameter 0) (color 0 0 0 0)
+  )
+  (junction (at 273.05 85.09) (diameter 0) (color 0 0 0 0)
+  )
+  (junction (at 195.58 22.86) (diameter 0) (color 0 0 0 0)
+  )
+  (junction (at 48.26 67.31) (diameter 0) (color 0 0 0 0)
+  )
+  (junction (at 119.38 54.61) (diameter 0) (color 0 0 0 0)
+  )
+  (junction (at 69.85 62.23) (diameter 0) (color 0 0 0 0)
   )
   (junction (at 273.05 111.76) (diameter 0) (color 0 0 0 0)
-  )
-  (junction (at 87.63 59.69) (diameter 0) (color 0 0 0 0)
-  )
-  (junction (at 48.26 67.31) (diameter 0) (color 0 0 0 0)
-  )
-  (junction (at 69.85 69.85) (diameter 0) (color 0 0 0 0)
-  )
-  (junction (at 44.45 59.69) (diameter 0) (color 0 0 0 0)
-  )
-  (junction (at 233.68 29.21) (diameter 0) (color 0 0 0 0)
-  )
-  (junction (at 69.85 67.31) (diameter 0) (color 0 0 0 0)
-  )
-  (junction (at 243.84 58.42) (diameter 0) (color 0 0 0 0)
-  )
-  (junction (at 139.7 22.86) (diameter 0) (color 0 0 0 0)
-  )
-  (junction (at 237.49 109.22) (diameter 0) (color 0 0 0 0)
-  )
-  (junction (at 107.95 82.55) (diameter 0) (color 0 0 0 0)
-  )
-  (junction (at 69.85 64.77) (diameter 0) (color 0 0 0 0)
-  )
-  (junction (at 44.45 67.31) (diameter 0) (color 0 0 0 0)
-  )
-  (junction (at 82.55 149.86) (diameter 0) (color 0 0 0 0)
-  )
-  (junction (at 100.33 82.55) (diameter 0) (color 0 0 0 0)
-  )
-  (junction (at 48.26 77.47) (diameter 0) (color 0 0 0 0)
-  )
-  (junction (at 232.41 144.78) (diameter 0) (color 0 0 0 0)
-  )
-  (junction (at 195.58 97.79) (diameter 0) (color 0 0 0 0)
-  )
-  (junction (at 82.55 160.02) (diameter 0) (color 0 0 0 0)
-  )
-  (junction (at 237.49 82.55) (diameter 0) (color 0 0 0 0)
-  )
-  (junction (at 273.05 85.09) (diameter 0) (color 0 0 0 0)
-  )
-  (junction (at 195.58 22.86) (diameter 0) (color 0 0 0 0)
-  )
-  (junction (at 119.38 54.61) (diameter 0) (color 0 0 0 0)
-  )
-  (junction (at 69.85 62.23) (diameter 0) (color 0 0 0 0)
   )
   (junction (at 92.71 62.23) (diameter 0) (color 0 0 0 0)
@@
     (stroke (width 0) (type default))
   )
-  (wire (pts (xy 48.26 71.12) (xy 48.26 67.31))
+  (wire (pts (xy 50.8 71.12) (xy 50.8 67.31))
     (stroke (width 0) (type default))
   )
@@
     (stroke (width 0) (type default))
   )
+  (wire (pts (xy 270.51 111.76) (xy 273.05 111.76))
+    (stroke (width 0) (type default))
+  )
   (wire (pts (xy 44.45 59.69) (xy 50.8 59.69))
     (stroke (width 0) (type default))
@@
     (stroke (width 0) (type default))
   )
-  (wire (pts (xy 55.88 76.2) (xy 55.88 77.47))
+  (wire (pts (xy 58.42 76.2) (xy 58.42 77.47))
     (stroke (width 0) (type default))
   )
@@
   )
   (wire (pts (xy 38.1 74.93) (xy 31.75 74.93))
-    (stroke (width 0) (type default))
-  )
-  (wire (pts (xy 269.24 111.76) (xy 270.51 111.76))
     (stroke (width 0) (type default))
   )
@@
     (stroke (width 0) (type default))
   )
-  (wire (pts (xy 48.26 77.47) (xy 55.88 77.47))
+  (wire (pts (xy 50.8 77.47) (xy 58.42 77.47))
     (stroke (width 0) (type default))
   )
@@
     (stroke (width 0) (type dash))
   )
-  (wire (pts (xy 48.26 76.2) (xy 48.26 77.47))
+  (wire (pts (xy 50.8 76.2) (xy 50.8 77.47))
     (stroke (width 0) (type default))
   )
@@
   )
   (wire (pts (xy 87.63 59.69) (xy 127 59.69))
+    (stroke (width 0) (type default))
+  )
+  (wire (pts (xy 48.26 67.31) (xy 50.8 67.31))
     (stroke (width 0) (type default))
   )
@@
     (stroke (width 0) (type default))
   )
-  (wire (pts (xy 48.26 77.47) (xy 48.26 78.74))
-    (stroke (width 0) (type default))
-  )
-  (wire (pts (xy 55.88 71.12) (xy 55.88 67.31))
+  (wire (pts (xy 50.8 77.47) (xy 50.8 78.74))
+    (stroke (width 0) (type default))
+  )
+  (wire (pts (xy 58.42 71.12) (xy 58.42 67.31))
     (stroke (width 0) (type default))
   )
@@
     (stroke (width 0) (type default))
   )
-  (wire (pts (xy 55.88 67.31) (xy 48.26 67.31))
+  (wire (pts (xy 58.42 67.31) (xy 50.8 67.31))
     (stroke (width 0) (type default))
   )
@@
   )
   (wire (pts (xy 100.33 82.55) (xy 102.87 82.55))
-    (stroke (width 0) (type default))
-  )
-  (wire (pts (xy 270.51 111.76) (xy 273.05 111.76))
     (stroke (width 0) (type default))
   )
@@
     )
   )
-  (symbol (lib_id "Device:C_Polarized_Small") (at 48.26 73.66 0) (unit 1)
-    (exclude_from_sim no) (in_bom yes) (on_board yes) (dnp no)
-    (property "Reference" "C9" (at 50.4952 72.4916 0)
-      (effects (font (size 1.27 1.27)) (justify left))
-    )
-    (property "Value" "100uF" (at 39.878 73.66 0)
-      (effects (font (size 1.27 1.27)) (justify left))
-    )
-    (property "Footprint" "Capacitor_SMD:CP_Elec_6.3x7.7" (at 48.26 73.66 0)
-      (effects (font (size 1.27 1.27)) (hide yes))
-    )
-    (property "Datasheet" "~" (at 48.26 73.66 0)
-      (effects (font (size 1.27 1.27)) (hide yes))
-    )
-    (property "Description" "Polarized capacitor, small symbol" (at 48.26 73.66 0)
+  (symbol (lib_id "Device:C_Polarized_Small") (at 50.8 73.66 0) (unit 1)
+    (exclude_from_sim no) (in_bom yes) (on_board yes) (dnp no)
+    (property "Reference" "C9" (at 53.0352 72.4916 0)
+      (effects (font (size 1.27 1.27)) (justify left))
+    )
+    (property "Value" "100uF" (at 42.418 73.66 0)
+      (effects (font (size 1.27 1.27)) (justify left))
+    )
+    (property "Footprint" "Capacitor_SMD:CP_Elec_6.3x7.7" (at 50.8 73.66 0)
+      (effects (font (size 1.27 1.27)) (hide yes))
+    )
+    (property "Datasheet" "~" (at 50.8 73.66 0)
+      (effects (font (size 1.27 1.27)) (hide yes))
+    )
+    (property "Description" "Polarized capacitor, small symbol" (at 50.8 73.66 0)
       (effects (font (size 1.27 1.27)) (hide yes))
     )
@@
     )
   )
-  (symbol (lib_id "Device:C_Polarized_Small") (at 55.88 73.66 0) (unit 1)
-    (exclude_from_sim no) (in_bom yes) (on_board yes) (dnp no)
-    (property "Reference" "C10" (at 59.182 72.898 0)
-      (effects (font (size 1.27 1.27)))
-    )
-    (property "Value" "10uF" (at 55.88 83.312 0)
-      (effects (font (size 1.27 1.27)))
-    )
-    (property "Footprint" "Capacitor_SMD:CP_Elec_6.3x5.8" (at 55.88 73.66 0)
-      (effects (font (size 1.27 1.27)) (hide yes))
-    )
-    (property "Datasheet" "~" (at 55.88 73.66 0)
-      (effects (font (size 1.27 1.27)) (hide yes))
-    )
-    (property "Description" "Polarized capacitor, small symbol" (at 55.88 73.66 0)
+  (symbol (lib_id "Device:C_Polarized_Small") (at 58.42 73.66 0) (unit 1)
+    (exclude_from_sim no) (in_bom yes) (on_board yes) (dnp no)
+    (property "Reference" "C10" (at 61.722 72.898 0)
+      (effects (font (size 1.27 1.27)))
+    )
+    (property "Value" "10uF" (at 58.42 83.312 0)
+      (effects (font (size 1.27 1.27)))
+    )
+    (property "Footprint" "Capacitor_SMD:CP_Elec_6.3x5.8" (at 58.42 73.66 0)
+      (effects (font (size 1.27 1.27)) (hide yes))
+    )
+    (property "Datasheet" "~" (at 58.42 73.66 0)
+      (effects (font (size 1.27 1.27)) (hide yes))
+    )
+    (property "Description" "Polarized capacitor, small symbol" (at 58.42 73.66 0)
       (effects (font (size 1.27 1.27)) (hide yes))
     )
@@
     )
   )
-  (symbol (lib_id "power:GND") (at 48.26 78.74 0) (unit 1)
+  (symbol (lib_id "power:GND") (at 50.8 78.74 0) (unit 1)
     (exclude_from_sim no) (in_bom yes) (on_board yes) (dnp no) (fields_autoplaced)
-    (property "Reference" "#PWR017" (at 48.26 85.09 0)
-      (effects (font (size 1.27 1.27)) (hide yes))
-    )
-    (property "Value" "GND" (at 48.26 83.82 0)
-      (effects (font (size 1.27 1.27)))
-    )
-    (property "Footprint" "" (at 48.26 78.74 0)
-      (effects (font (size 1.27 1.27)) (hide yes))
-    )
-    (property "Datasheet" "" (at 48.26 78.74 0)
-      (effects (font (size 1.27 1.27)) (hide yes))
-    )
-    (property "Description" "Power symbol creates a global label with name \"GND\" , ground" (at 48.26 78.74 0)
-      (effects (font (size 1.27 1.27)) (hide yes))
-    )
+    (property "Reference" "#PWR017" (at 50.8 85.09 0)
+      (effects (font (size 1.27 1.27)) (hide yes))
+    )
+    (property "Value" "GND" (at 50.8 83.82 0)
+      (effects (font (size 1.27 1.27)))
+    )
+    (property "Footprint" "" (at 50.8 78.74 0)
+      (effects (font (size 1.27 1.27)) (hide yes))
+    )
+    (property "Datasheet" "" (at 50.8 78.74 0)
+      (effects (font (size 1.27 1.27)) (hide yes))
+    )
+    (property "Description" "Power symbol creates a global label with name \"GND\" , ground" (at 50.8 78.74 0)
+      (effects (font (size 1.27 1.27)) (hide yes))
+    )

Commit message: Deploying to main from @ electrified/rcbus-opl3@b421ed74cec5974dc3bbc62da0d3b0773d89e203 🚀
Parts:
- C1: Farnell url (none) -> https://uk.farnell.com/wurth-elektronik/875105240001/cap-10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; MPN (none) -> 875105240001
- C10, C2, C7: Farnell url (none) -> https://uk.farnell.com/wurth-elektronik/875105240001/cap-10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
- C3: Farnell url (none) -> https://uk.farnell.com/multicomp-pro/mc0603n272j500ct/cap-m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
- C9: Farnell url (none) -> https://uk.farnell.com/kemet/a768eb107m1elas036/cap-100uf-2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
- R10, R11, R6, R7, R8, R9: Farnell url (none) -> https://uk.farnell.com/multicomp-pro/mcwr06x1002ftl/res-10k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
- U3: Farnell url (none) -> https://uk.farnell.com/texas-instruments/cd74hct688m96/comp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
- Y1: Farnell url (none) -> https://uk.farnell.com/multicomp-pro/mcsjk-6nc1-14-31818-25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
Changed lines of the file:
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@@
       (effects (font (size 1.27 1.27)) (hide yes))
     )
-    (property "Description" "Polarized capacitor, small symbol" (at 50.8 73.66 0)
+    (property "Description" "Polymer Aluminium Electrolytic Capacitor, 100 µF, 25 V, Radial Can - SMD, 0.036 ohm" (at 50.8 73.66 0)
+      (effects (font (size 1.27 1.27)) (hide yes))
+    )
+    (property "Farnell url" "https://uk.farnell.com/kemet/a768eb107m1elas036/cap-100uf-25v-alu-elec-smd-polymer/dp/4071180" (at 50.8 73.66 0)
       (effects (font (size 1.27 1.27)) (hide yes))
     )
@@
       (effects (font (size 1.27 1.27)) (hide yes))
     )
-    (property "Description" "8-bit magnitude comparator" (at 139.7 59.69 0)
+    (property "Description" "Digital Comparator, 74HCT688, Magnitude, 8 Channels, 8bit, SOIC, 20 Pins" (at 139.7 59.69 0)
+      (effects (font (size 1.27 1.27)) (hide yes))
+    )
+    (property "Farnell url" "https://uk.farnell.com/texas-instruments/cd74hct688m96/comparator-magnitude-8bit-soic/dp/3006842" (at 139.7 59.69 0)
       (effects (font (size 1.27 1.27)) (hide yes))
     )
@@
       (effects (font (size 1.27 1.27)) (hide yes))
     )
-    (property "Datasheet" "~" (at 233.68 33.02 0)
-      (effects (font (size 1.27 1.27)) (hide yes))
-    )
-    (property "Description" "Polarized capacitor, small symbol" (at 233.68 33.02 0)
+    (property "Datasheet" "https://www.we-online.com/components/products/datasheet/875105240001.pdf" (at 233.68 33.02 0)
+      (effects (font (size 1.27 1.27)) (hide yes))
+    )
+    (property "Description" "Polymer Aluminium Electrolytic Capacitor, 10 µF, 10 V, Radial Can - SMD, 0.045 ohm" (at 233.68 33.02 0)
+      (effects (font (size 1.27 1.27)) (hide yes))
+    )
+    (property "Farnell url" "https://uk.farnell.com/wurth-elektronik/875105240001/cap-10-f-10v-20/dp/2466639" (at 233.68 33.02 0)
+      (effects (font (size 1.27 1.27)) (hide yes))
+    )
+    (property "MPN" "875105240001" (at 233.68 33.02 0)
       (effects (font (size 1.27 1.27)) (hide yes))
     )
@@
       (effects (font (size 1.27 1.27)) (hide yes))
     )
-    (property "Datasheet" "~" (at 199.39 132.08 0)
-      (effects (font (size 1.27 1.27)) (hide yes))
-    )
-    (property "Description" "Polarized capacitor, small symbol" (at 199.39 132.08 0)
+    (property "Datasheet" "https://www.we-online.com/components/products/datasheet/875105240001.pdf" (at 199.39 132.08 0)
+      (effects (font (size 1.27 1.27)) (hide yes))
+    )
+    (property "Description" "Polymer Aluminium Electrolytic Capacitor, 10 µF, 10 V, Radial Can - SMD, 0.045 ohm" (at 199.39 132.08 0)
+      (effects (font (size 1.27 1.27)) (hide yes))
+    )
+    (property "Farnell url" "https://uk.farnell.com/wurth-elektronik/875105240001/cap-10-f-10v-20/dp/2466639" (at 199.39 132.08 0)
       (effects (font (size 1.27 1.27)) (hide yes))
     )
@@
       (effects (font (size 1.27 1.27)) (hide yes))
     )
-    (property "Description" "Resistor, small symbol" (at 97.79 78.74 0)
+    (property "Description" "SMD Chip Resistor, 10 kohm, ± 1%, 100 mW, 0603 [1608 Metric], Thick Film, General Purpose" (at 97.79 78.74 0)
+      (effects (font (size 1.27 1.27)) (hide yes))
+    )
+    (property "Farnell url" "https://uk.farnell.com/multicomp-pro/mcwr06x1002ftl/res-10k-1-0-1w-0603-thick-film/dp/2447230" (at 97.79 78.74 0)
       (effects (font (size 1.27 1.27)) (hide yes))
     )
@@
       (effects (font (size 1.27 1.27)) (hide yes))
     )
-    (property "Description" "Resistor, small symbol" (at 113.03 78.74 0)
+    (property "Description" "SMD Chip Resistor, 10 kohm, ± 1%, 100 mW, 0603 [1608 Metric], Thick Film, General Purpose" (at 113.03 78.74 0)
+      (effects (font (size 1.27 1.27)) (hide yes))
+    )
+    (property "Farnell url" "https://uk.farnell.com/multicomp-pro/mcwr06x1002ftl/res-10k-1-0-1w-0603-thick-film/dp/2447230" (at 113.03 78.74 0)
       (effects (font (size 1.27 1.27)) (hide yes))
     )
@@
       (effects (font (size 1.27 1.27)) (hide yes))
     )
-    (property "Description" "Resistor, small symbol" (at 87.63 78.74 0)
+    (property "Description" "SMD Chip Resistor, 10 kohm, ± 1%, 100 mW, 0603 [1608 Metric], Thick Film, General Purpose" (at 87.63 78.74 0)
+      (effects (font (size 1.27 1.27)) (hide yes))
+    )
+    (property "Farnell url" "https://uk.farnell.com/multicomp-pro/mcwr06x1002ftl/res-10k-1-0-1w-0603-thick-film/dp/2447230" (at 87.63 78.74 0)
       (effects (font (size 1.27 1.27)) (hide yes))
     )
@@
       (effects (font (size 1.27 1.27)) (hide yes))
     )
-    (property "Description" "Resistor, small symbol" (at 107.95 78.74 0)
+    (property "Description" "SMD Chip Resistor, 10 kohm, ± 1%, 100 mW, 0603 [1608 Metric], Thick Film, General Purpose" (at 107.95 78.74 0)
+      (effects (font (size 1.27 1.27)) (hide yes))
+    )
+    (property "Farnell url" "https://uk.farnell.com/multicomp-pro/mcwr06x1002ftl/res-10k-1-0-1w-0603-thick-film/dp/2447230" (at 107.95 78.74 0)
       (effects (font (size 1.27 1.27)) (hide yes))
     )
@@
       (effects (font (size 1.27 1.27)) (hide yes))
     )
-    (property "Datasheet" "~" (at 58.42 73.66 0)
-      (effects (font (size 1.27 1.27)) (hide yes))
-    )
-    (property "Description" "Polarized capacitor, small symbol" (at 58.42 73.66 0)
+    (property "Datasheet" "https://www.we-online.com/components/products/datasheet/875105240001.pdf" (at 58.42 73.66 0)
+      (effects (font (size 1.27 1.27)) (hide yes))
+    )
+    (property "Description" "Polymer Aluminium Electrolytic Capacitor, 10 µF, 10 V, Radial Can - SMD, 0.045 ohm" (at 58.42 73.66 0)
+      (effects (font (size 1.27 1.27)) (hide yes))
+    )
+    (property "Farnell url" "https://uk.farnell.com/wurth-elektronik/875105240001/cap-10-f-10v-20/dp/2466639" (at 58.42 73.66 0)
       (effects (font (size 1.27 1.27)) (hide yes))
     )
@@
       (effects (font (size 1.27 1.27)) (hide yes))
     )
-    (property "Description" "Resistor, small symbol" (at 92.71 78.74 0)
+    (property "Description" "SMD Chip Resistor, 10 kohm, ± 1%, 100 mW, 0603 [1608 Metric], Thick Film, General Purpose" (at 92.71 78.74 0)
+      (effects (font (size 1.27 1.27)) (hide yes))
+    )
+    (property "Farnell url" "https://uk.farnell.com/multicomp-pro/mcwr06x1002ftl/res-10k-1-0-1w-0603-thick-film/dp/2447230" (at 92.71 78.74 0)
       (effects (font (size 1.27 1.27)) (hide yes))
     )
@@
       (effects (font (size 1.27 1.27)) (hide yes))
     )
-    (property "Datasheet" "http://www.abracon.com/Oscillators/ASV.pdf" (at 80.01 167.64 0)
-      (effects (font (size 1.27 1.27)) (hide yes))
-    )
-    (property "Description" "3.3V HCMOS SMD Crystal Clock Oscillator, Abracon" (at 82.55 167.64 0)
+    (property "Datasheet" "https://4donline.ihs.com/images/VipMasterIC/IC/SCMP/SCMP-S-A0010069830/SCMP-S-A0010069830-1.pdf?hkey=6D3A4C79FDBF58556ACFDE234799DDF0" (at 80.01 167.64 0)
+      (effects (font (size 1.27 1.27)) (hide yes))
+    )
+    (property "Description" "Oscillator, 14.31818 MHz, 25 ppm, SMD, 7mm x 5mm, CMOS / TTL, 5 V" (at 82.55 167.64 0)
+      (effects (font (size 1.27 1.27)) (hide yes))
+    )
+    (property "Farnell url" "https://uk.farnell.com/multicomp-pro/mcsjk-6nc1-14-31818-25-b/oscillator-14-31818mhz-7mm-x-5mm/dp/2854363" (at 82.55 167.64 0)
       (effects (font (size 1.27 1.27)) (hide yes))
     )
@@
       (effects (font (size 1.27 1.27)) (hide yes))
     )
-    (property "Datasheet" "" (at 195.58 80.518 0)
-      (effects (font (size 1.27 1.27)) (hide yes))
-    )
-    (property "Description" "" (at 195.58 78.486 0)
+    (property "Datasheet" "https://www.ardent-tool.com/datasheets/Yamaha_YAC512.pdf" (at 195.58 80.518 0)
+      (effects (font (size 1.27 1.27)) (hide yes))
+    )
+    (property "Description" "2-Channel floating D/A converter" (at 195.58 78.486 0)
       (effects (font (size 1.27 1.27)) (hide yes))
     )
@@
       (effects (font (size 1.27 1.27)) (hide yes))
     )
-    (property "Datasheet" "" (at 119.38 164.338 0)
+    (property "Datasheet" "http://www.bitsavers.org/components/yamaha/YMF262_199110.pdf" (at 119.38 164.338 0)
       (effects (font (size 1.27 1.27)) (hide yes))
     )
@@
       (effects (font (size 1.27 1.27)) (hide yes))
     )
+    (property "Farnell url" "https://uk.farnell.com/multicomp-pro/mc0603n272j500ct/cap-mlcc-2700pf-c0g-np0-50v-0603/dp/4540299" (at 237.49 85.09 0)
+      (effects (font (size 1.27 1.27)) (hide yes))
+    )
     (pin "1")
     (pin "2")
@@
       (effects (font (size 1.27 1.27)) (hide yes))
     )
-    (property "Datasheet" "~" (at 199.39 152.4 0)
-      (effects (font (size 1.27 1.27)) (hide yes))
-    )
-    (property "Description" "Polarized capacitor, small symbol" (at 199.39 152.4 0)
+    (property "Datasheet" "https://www.we-online.com/components/products/datasheet/875105240001.pdf" (at 199.39 152.4 0)
+      (effects (font (size 1.27 1.27)) (hide yes))
+    )
+    (property "Description" "Polymer Aluminium Electrolytic Capacitor, 10 µF, 10 V, Radial Can - SMD, 0.045 ohm" (at 199.39 152.4 0)
+      (effects (font (size 1.27 1.27)) (hide yes))
+    )
+    (property "Farnell url" "https://uk.farnell.com/wurth-elektronik/875105240001/cap-10-f-10v-20/dp/2466639" (at 199.39 152.4 0)
       (effects (font (size 1.27 1.27)) (hide yes))
     )
@@
       (effects (font (size 1.27 1.27)) (hide yes))
     )
-    (property "Description" "Resistor, small symbol" (at 102.87 78.74 0)
-      (effects (font (size 1.27 1.27)) (hide yes))
-    )
+    (property "Description" "SMD Chip Resistor, 10 kohm, ± 1%, 100 mW, 0603 [1608 Metric], Thick Film, General Purpose" (at 102.87 78.74 0)
+      (effects (font (size 1.27 1.27)) (hide yes))
+    )
+    (property "Farnell url" "https://uk.farnell.com/multicomp-pro/mcwr06x1002ftl/res-10k-1-0-1w-0603-thick-film/dp/2447230" (at 102.87 78.74 0)
+      (effects (font (size 1.27 1.27)) (hide yes))
+    )
