File: Browse/rcbus-opl3.kicad_sch (KiCad schematic)
At the start: 33 parts, among them CON1 3.5mm jack, P1 RC2014 BUS, U1 TL074, U2 YAC512, U3 74HCT688, U4 YMF262, Y1 14.3181MHz

Commit message: Deploying to main from @ electrified/rcbus-opl3@75fd01174487a1f644e8e46dc09a2a87611ef887 🚀
Parts:
- C1: Farnell url https://uk.farnell.com/wurth-elektronik/875105240001/cap-10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 -> (none); Farnell_URI (none) -> https://uk.farnell.com/wurth-elektronik/875105240001/cap-10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; MPN 875105240001 -> (none)
- C10, C2, C7: Farnell url https://uk.farnell.com/wurth-elektronik/875105240001/cap-10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 -> (none); Farnell_URI (none) -> https://uk.farnell.com/wurth-elektronik/875105240001/cap-10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
- C11, C12, C13, C5, C8: Farnell_URI (none) -> https://uk.farnell.com/multicomp-pro/mc0603b104m250ct/cap-0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
- C3: Farnell url https://uk.farnell.com/multicomp-pro/mc0603n272j500ct/cap-m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 -> (none); Farnell_URI (none) -> https://uk.farnell.com/multicomp-pro/mc0603n272j500ct/cap-m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
- C4: Farnell_URI (none) -> https://uk.farnell.com/multicomp-pro/mc0603n272j500ct/cap-m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
- C6: Farnell_URI (none) -> https://uk.farnell.com/multicomp-pro/mc0603n680j500ct/cap-6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
- C9: Farnell url https://uk.farnell.com/kemet/a768eb107m1elas036/cap-100uf-2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 -> (none); Farnell_URI (none) -> https://uk.farnell.com/kemet/a768eb107m1elas036/cap-100uf-2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
- CON1: Category Connectors, Interconnects -> (none); DK_Datasheet_Link https://www.cui.com/product/resource/digikeypdf/sj1-352xn_s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 -> (none); DK_Detail_Page /product-detail/en/cui-inc/SJ1-3523N/CP1-3523N-ND/738689 -> (none); Digi-Key_PN CP1-3523N-ND -> (none); Family Barrel - Audio Connectors -> (none); Farnell_URI (none) -> https://uk.farnell.com/cliff-electronic-components/fc68131/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; MPN SJ1-3523N -> (none); Manufacturer CUI Inc. -> (none); Status Active -> (none)
- JP1: Farnell_URI (none) -> https://uk.farnell.com/harwin/m20-9980346/connector-header-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
- P1: Farnell_URI (none) -> https://uk.farnell.com/wurth-elektronik/61304011021/header-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
- R1: Farnell_URI (none) -> https://uk.farnell.com/multicomp-pro/mcwr06x33r0ftl/res-33r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
- R10, R11, R6, R7, R8, R9: Farnell url https://uk.farnell.com/multicomp-pro/mcwr06x1002ftl/res-10k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 -> (none); Farnell_URI (none) -> https://uk.farnell.com/multicomp-pro/mcwr06x1002ftl/res-10k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
- R2, R5: Farnell_URI (none) -> https://uk.farnell.com/multicomp-pro/mcwr06x1002ftl/res-10k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
- R3, R4: Farnell_URI (none) -> https://uk.farnell.com/multicomp-pro/mcwr06x1000ftl/res-100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
- U1: Farnell_URI (none) -> https://uk.farnell.com/stmicroelectronics/tl074cdt/opamp-3m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
- U3: Farnell url https://uk.farnell.com/texas-instruments/cd74hct688m96/comp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 -> (none); Farnell_URI (none) -> https://uk.farnell.com/texas-instruments/cd74hct688m96/comp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
- Y1: Farnell url https://uk.farnell.com/multicomp-pro/mcsjk-6nc1-14-31818-25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 -> (none); Farnell_URI (none) -> https://uk.farnell.com/multicomp-pro/mcsjk-6nc1-14-31818-25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
Other:
- moved on the sheet: C2, C7, CON1, R2, R3, R4, R5
