File: Browse/rcbus-opl3.kicad_sch (KiCad schematic)
At the start: 33 parts, among them CON1 3.5mm jack, P1 RC2014 BUS, U1 TL074, U2 YAC512, U3 74HCT688, U4 YMF262, Y1 14.3181MHz

Commit message: Deploying to main from @ electrified/rcbus-opl3@ddbdba2873f61b31b89cbd436bb303ada35639e9 🚀
Parts:
- C1, C10, C2, C7: Farnell_URI https://uk.farnell.com/wurth-elektronik/875105240001/cap-10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 -> https://uk.farnell.com/kemet/edk106m035a9baa/cap-10uf-35v-a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; MPN (none) -> EDK106M035A9BAA
- C11, C12, C13, C5, C8: MPN (none) -> MC0603B104M250CT
- C3, C4: MPN (none) -> MC0603N272J500CT
- C6: MPN (none) -> MC0603N680J500CT
- C9: Farnell_URI https://uk.farnell.com/kemet/a768eb107m1elas036/cap-100uf-2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 -> https://uk.farnell.com/kemet/edk107m035a9haa/cap-100-f-35v-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; MPN (none) -> EDK107M035A9HAA
- CON1: MPN (none) -> FC68131
- JP1: value BASE ADDRESS -> 2x06 pin header; MPN (none) -> M20-9980346
- P1: value RC2014 BUS -> 1x39 pin header; MPN (none) -> 61304011021
- R1: MPN (none) -> MCWR06X33R0FTL
- R10, R11, R2, R5, R6, R7, R8, R9: MPN (none) -> MCWR06X1002FTL
- R3, R4: MPN (none) -> MCWR06X1000FTL
- U1: MPN (none) -> TL074CDT
- U3: MPN (none) -> CD74HCT688M96
- Y1: MPN (none) -> MCSJK-6NC1-14.31818-25-B

Commit message: Deploying to main from @ electrified/rcbus-opl3@4d7316e7b421a6980499a84c96f6f3c4ba9db318 🚀
Parts:
- C1, C10, C2, C7: footprint Capacitor_SMD:CP_Elec_6.3x5.8 -> Capacitor_SMD:CP_Elec_4x5.4
- U2: footprint Package_SO:SOP-16_4.55x10.3mm_P1.27mm -> Package_SO:SOIC-16W_5.3x10.2mm_P1.27mm
- U4: footprint Package_SO:SOP-24_7.5x15.4mm_P1.27mm -> electrified:SOP-24_wider
Changed lines of the file:
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@@
   (junction (at 97.79 82.55) (diameter 0) (color 0 0 0 0)
   )
-  (junction (at 255.27 43.18) (diameter 0) (color 0 0 0 0)
-  )
   (junction (at 87.63 59.69) (diameter 0) (color 0 0 0 0)
   )
@@
   )
   (junction (at 218.44 149.86) (diameter 0) (color 0 0 0 0)
+  )
+  (junction (at 251.46 43.18) (diameter 0) (color 0 0 0 0)
   )
   (junction (at 232.41 149.86) (diameter 0) (color 0 0 0 0)
@@
     (stroke (width 0) (type default))
   )
-  (wire (pts (xy 255.27 43.18) (xy 255.27 45.72))
-    (stroke (width 0) (type default))
-  )
   (polyline (pts (xy 62.23 99.06) (xy 62.23 186.69))
     (stroke (width 0) (type dash))
@@
     (stroke (width 0) (type default))
   )
+  (wire (pts (xy 251.46 34.29) (xy 255.27 34.29))
+    (stroke (width 0) (type default))
+  )
   (wire (pts (xy 119.38 52.07) (xy 127 52.07))
     (stroke (width 0) (type default))
@@
     (stroke (width 0) (type default))
   )
-  (wire (pts (xy 248.92 123.19) (xy 248.92 114.3))
+  (wire (pts (xy 251.46 123.19) (xy 251.46 114.3))
     (stroke (width 0) (type default))
   )
@@
     (stroke (width 0) (type default))
   )
-  (wire (pts (xy 248.92 96.52) (xy 273.05 96.52))
+  (wire (pts (xy 251.46 96.52) (xy 273.05 96.52))
     (stroke (width 0) (type default))
   )
@@
     (stroke (width 0) (type default))
   )
-  (wire (pts (xy 207.01 43.18) (xy 255.27 43.18))
+  (wire (pts (xy 207.01 43.18) (xy 251.46 43.18))
     (stroke (width 0) (type default))
   )
@@
     (stroke (width 0) (type default))
   )
-  (wire (pts (xy 248.92 123.19) (xy 273.05 123.19))
+  (wire (pts (xy 251.46 123.19) (xy 273.05 123.19))
     (stroke (width 0) (type default))
   )
@@
     (stroke (width 0) (type default))
   )
-  (wire (pts (xy 273.05 31.75) (xy 273.05 45.72))
+  (wire (pts (xy 273.05 31.75) (xy 273.05 43.18))
     (stroke (width 0) (type default))
   )
@@
     (stroke (width 0) (type default))
   )
-  (wire (pts (xy 248.92 87.63) (xy 255.27 87.63))
+  (wire (pts (xy 251.46 87.63) (xy 255.27 87.63))
     (stroke (width 0) (type default))
   )
@@
     (stroke (width 0) (type default))
   )
-  (wire (pts (xy 255.27 34.29) (xy 255.27 43.18))
+  (wire (pts (xy 251.46 34.29) (xy 251.46 43.18))
     (stroke (width 0) (type default))
   )
@@
     (stroke (width 0) (type default))
   )
-  (wire (pts (xy 273.05 45.72) (xy 255.27 45.72))
+  (wire (pts (xy 273.05 43.18) (xy 251.46 43.18))
     (stroke (width 0) (type default))
   )
@@
     (stroke (width 0) (type default))
   )
-  (wire (pts (xy 248.92 96.52) (xy 248.92 87.63))
+  (wire (pts (xy 251.46 96.52) (xy 251.46 87.63))
     (stroke (width 0) (type default))
   )
@@
     (stroke (width 0) (type default))
   )
-  (wire (pts (xy 248.92 114.3) (xy 255.27 114.3))
+  (wire (pts (xy 251.46 114.3) (xy 255.27 114.3))
     (stroke (width 0) (type default))
   )
@@
       (effects (font (size 1.27 1.27)) (justify left))
     )
-    (property "Footprint" "Capacitor_SMD:CP_Elec_6.3x5.8" (at 233.68 33.02 0)
+    (property "Footprint" "Capacitor_SMD:CP_Elec_4x5.4" (at 233.68 33.02 0)
       (effects (font (size 1.27 1.27)) (hide yes))
     )
@@
       (effects (font (size 1.27 1.27)))
     )
-    (property "Footprint" "Capacitor_SMD:CP_Elec_6.3x5.8" (at 199.39 134.62 0)
+    (property "Footprint" "Capacitor_SMD:CP_Elec_4x5.4" (at 199.39 134.62 0)
       (effects (font (size 1.27 1.27)) (hide yes))
     )
@@
       (effects (font (size 1.27 1.27)))
     )
-    (property "Footprint" "Capacitor_SMD:CP_Elec_6.3x5.8" (at 58.42 73.66 0)
+    (property "Footprint" "Capacitor_SMD:CP_Elec_4x5.4" (at 58.42 73.66 0)
       (effects (font (size 1.27 1.27)) (hide yes))
     )
@@
       (effects (font (size 1.27 1.27)) (justify left))
     )
-    (property "Footprint" "Package_SO:SOP-16_4.55x10.3mm_P1.27mm" (at 195.326 97.282 0)
+    (property "Footprint" "Package_SO:SOIC-16W_5.3x10.2mm_P1.27mm" (at 195.326 97.282 0)
       (effects (font (size 1.27 1.27)) (hide yes))
     )
@@
       (effects (font (size 1.27 1.27)) (justify left))
     )
-    (property "Footprint" "Package_SO:SOP-24_7.5x15.4mm_P1.27mm" (at 119.126 181.102 0)
+    (property "Footprint" "electrified:SOP-24_wider" (at 119.126 181.102 0)
       (effects (font (size 1.27 1.27)) (hide yes))
     )
@@
       (effects (font (size 1.27 1.27)))
     )
-    (property "Footprint" "Capacitor_SMD:CP_Elec_6.3x5.8" (at 199.39 149.86 0)
-      (effects (font (size 1.27 1.27)) (hide yes))
-    )
+    (property "Footprint" "Capacitor_SMD:CP_Elec_4x5.4" (at 199.39 149.86 0)
+      (effects (font (size 1.27 1.27)) (hide yes))
+    )

Commit message: Deploying to main from @ electrified/rcbus-opl3@4b95d9054967e44d5d8dd23a98a17ec64137cdb5 🚀
Parts:
- U2: footprint Package_SO:SOIC-16W_5.3x10.2mm_P1.27mm -> Package_SO:SOP-16_4.55x10.3mm_P1.27mm
