File: Browse/rcbus-opl3.kicad_pcb (KiCad board)
At the start: 2 copper layers, 100 x 50 mm, 38 parts, among them CON1 3.5mm jack, P1 1x39 pin header, U1 TL074, U2 YAC512, U3 74HCT688, U4 YMF262, Y1 14.3181MHz

Commit message: Deploying to main from @ electrified/rcbus-opl3@4d7316e7b421a6980499a84c96f6f3c4ba9db318 🚀
Parts:
- C1, C10, C2, C7: footprint Capacitor_SMD:CP_Elec_6.3x5.8 -> Capacitor_SMD:CP_Elec_4x5.4
- U2: footprint Package_SO:SOP-16_4.55x10.3mm_P1.27mm -> Package_SO:SOIC-16W_5.3x10.2mm_P1.27mm
- U4: footprint Package_SO:SOP-24_7.5x15.4mm_P1.27mm -> electrified:SOP-24_wider
- moved G2 1.27 mm to (93.8, 123.0)
Routing:
- net GND: track 32.7 -> 33.6 mm, vias 86 -> 85
Other:
- board text added: "RCBus OPL3 sound card"
- board text removed: "RCBus OPL3 Sound Card"

Commit message: Deploying to main from @ electrified/rcbus-opl3@5a83b2ec4dff658a1e33cbe5684ae3260741873a 🚀
Parts:
- moved C10 2.70 mm to (102.5, 148.2)
- moved C12 0.70 mm to (118.3, 142.4)
- moved C6 0.50 mm to (123.4, 128.7)
- moved R1 0.50 mm to (125.4, 128.7)
- moved CON1 0.43 mm to (149.0, 125.6)
Routing:
- net +5V: track 229.1 -> 226.3 mm
- net /D5: track 11.8 -> 14.1 mm
- net /D6: track 14.2 -> 16.0 mm
- net /D4: track 10.6 -> 12.3 mm
- net /D7: track 16.7 -> 18.0 mm
- net /R: track 14.1 -> 15.3 mm
- net /D3: track 9.59 -> 10.6 mm
- net Net-(U1B-+): track 8.26 -> 9.08 mm
- net /AUDIO_CH1: track 20.8 -> 21.6 mm
- net /DOAB: track 21.5 -> 22.3 mm
- net /L: track 21.7 -> 20.9 mm
- net /DAC_CLK: track 19.8 -> 20.6 mm
- net GND: track 33.6 -> 33.9 mm, vias 85 -> 84
Other:
- board text added: "▲"

Commit message: Deploying to main from @ electrified/rcbus-opl3@4b95d9054967e44d5d8dd23a98a17ec64137cdb5 🚀
Parts:
- U2: footprint Package_SO:SOIC-16W_5.3x10.2mm_P1.27mm -> Package_SO:SOP-16_4.55x10.3mm_P1.27mm
