File: Presentation/boards/rcbus-ymf262.kicad_pcb (KiCad board)
At the start: 2 copper layers, 100 x 50 mm, 43 parts, among them CON1 SJ1-3523N, P1 RC2014 BUS, U1 74HCT688, U2 YMF262, U3 YAC512, U4 TL074, Y1 SG-8002CA

Commit message: Deploying to main from @ electrified/rcbus-ymf262@9c8d0cd003b39a240463bae4e94c496cca633260 🚀
Parts:
- moved C16 9.41 mm to (132.0, 126.3)
- moved C18 9.41 mm to (142.3, 126.3)
- moved R11 9.41 mm to (137.1, 126.3)
- moved C5 6.84 mm to (96.2, 137.2), turned to 90 degrees
- moved C11 5.33 mm to (121.5, 131.4)
- moved L1 5.14 mm to (84.5, 137.1), turned to -90 degrees
- moved L2 5.00 mm to (93.0, 137.1), turned to 90 degrees
- moved C4 2.51 mm to (90.0, 137.2), turned to -90 degrees
- moved R7 1.00 mm to (123.2, 131.4)
- moved C2 0.51 mm to (82.0, 137.1), turned to 90 degrees
- moved C3 0.11 mm to (87.0, 137.1), turned to -90 degrees
Connections:
- C10 pad 1: /AUDIO_CH1 -> /AUDIO_CH2
- C13 pad 1: /L -> /R
- C14 pad 2: /R -> /L
- C9 pad 1: /AUDIO_CH2 -> /AUDIO_CH1
- R8 pad 2: /L -> /R
- R9 pad 2: /R -> /L
- U4 pad 10: /AUDIO_CH2 -> /AUDIO_CH1
- U4 pad 12: /AUDIO_CH1 -> /AUDIO_CH2
- U4 pad 14: /R -> /L
- U4 pad 8: /L -> /R
Routing:
- net GND: track 64.6 -> 34.7 mm
- net Net-(C18-Pad1): track 28.0 -> 14.5 mm
- net Net-(C3-Pad1): track 21.1 -> 8.93 mm, vias 3 -> 0
- net /L: track 18.1 -> 29.7 mm
- net /AUDIO_CH1: track 33.2 -> 22.7 mm
- net VCC: track 129.8 -> 125.3 mm
- net Net-(U3-AOUT): track 16.9 -> 12.6 mm
- net /AUDIO_CH2: track 20.9 -> 23.6 mm, vias 2 -> 0
- net /R: track 25.7 -> 23.0 mm
- net Net-(U4B--): track 5.58 -> 3.92 mm
- net Net-(JP1-Pin_1): track 28.7 -> 29.5 mm
- net +5VA: track 69.8 -> 70.4 mm, vias 1 -> 0
- net Net-(U3-SWIN): track 5.51 -> 6.14 mm
- net /~{CS}: track 51.7 -> 52.2 mm
- net Net-(JP1-Pin_7): track 28.1 -> 27.6 mm

Commit message: Deploying to main from @ electrified/rcbus-ymf262@646990f17bd25725641340863379bc60f4c51cf2 🚀
Parts:
- moved R6 0.15 mm to (74.2, 156.0)
- moved R3 0.15 mm to (74.2, 148.5)
- moved R5 0.15 mm to (74.2, 153.5)
- moved R4 0.15 mm to (74.2, 151.0)
- moved R2 0.06 mm to (74.2, 146.0)
Routing:
- net GND: track 34.7 -> 47.5 mm, vias 62 -> 68
- net VCC: track 125.3 -> 122.2 mm
- net Net-(JP1-Pin_1): track 29.5 -> 31.4 mm
- net /AUDIO_CH1: track 22.7 -> 24.6 mm
- net Net-(U3-MP): track 16.3 -> 17.9 mm
- net /A1: track 27.3 -> 28.5 mm
- net /~{IORQ}: track 52.4 -> 53.3 mm
- net Net-(JP1-Pin_9): track 30.6 -> 29.7 mm
- net /~{CS}: track 52.2 -> 53.0 mm
- net /AUDIO_CH2: track 23.6 -> 24.3 mm
- net /A0: track 23.0 -> 23.6 mm
- net Net-(JP1-Pin_7): track 27.6 -> 27.0 mm
