File: Presentation/boards/rcbus-opl3.kicad_pcb (KiCad board)
At the start: 2 copper layers, 100 x 50 mm, 39 parts, among them CON1 SJ1-3523N, P1 RC2014 BUS, U1 74HCT688, U2 YMF262, U3 YAC512, U4 TL074, Y1 SG-8002CA

Commit message: Deploying to main from @ electrified/rcbus-opl3@ca335f471b0cc053c0f7ada637c7f1deac17d0b8 🚀
Parts:
- removed C2: 10nF, Capacitor_SMD:C_0603_1608Metric
- removed C3: 100nF, Capacitor_SMD:C_0603_1608Metric
- removed C4: 10uF, Capacitor_SMD:C_1206_3216Metric
- removed L1: BLM18PG221SN1D, Inductor_SMD:L_0603_1608Metric
- removed L2: 33uH, Inductor_SMD:L_0603_1608Metric
- C15, C16: footprint Capacitor_SMD:CP_Elec_5x5.9 -> Capacitor_SMD:CP_Elec_6.3x5.8
- C5: value 10uF -> 100uF; footprint Capacitor_SMD:C_1206_3216Metric -> Capacitor_SMD:CP_Elec_6.3x7.7
- C8: footprint Capacitor_SMD:C_0603_1608Metric -> Capacitor_SMD:CP_Elec_6.3x5.8
- moved C5 18.4 mm to (98.5, 155.4), turned to -90 degrees
- moved C8 8.58 mm to (108.2, 131.8)
Connections:
- C1 pad 1: VCC -> +5V
- C12 pad 1: +5VA -> +5V
- C19 pad 1: VCC -> +5V
- C5 pad 1: +5VA -> +5V
- C6 pad 1: VCC -> +5V
- C7 pad 1: +5VA -> +5V
- JP1 pad 10: VCC -> +5V
- JP1 pad 12: VCC -> +5V
- JP1 pad 2: VCC -> +5V
- JP1 pad 4: VCC -> +5V
- JP1 pad 6: VCC -> +5V
- JP1 pad 8: VCC -> +5V
- P1 pad 18: VCC -> +5V
- U1 pad 20: VCC -> +5V
- U2 pad 1: VCC -> +5V
- U3 pad 1: +5VA -> +5V
- U3 pad 3: +5VA -> +5V
- U3 pad 6: +5VA -> +5V
- U3 pad 9: +5VA -> +5V
- U4 pad 4: +5VA -> +5V
- Y1 pad 1: VCC -> +5V
- Y1 pad 4: VCC -> +5V
Routing:
- net +5V: track 0.00 -> 178.2 mm, vias 0 -> 2
- net VCC: track 126.4 -> 0.00 mm, vias 2 -> 0
- net +5VA: track 70.5 -> 0.00 mm
- net Net-(U3-CV): track 12.2 -> 25.5 mm
- net Net-(C3-Pad1): track 8.93 -> 0.00 mm
- net GND: track 38.9 -> 31.6 mm, vias 35 -> 31
- net /~{CS}: track 54.9 -> 56.6 mm

Commit message: Deploying to main from @ electrified/rcbus-opl3@95905a1b3d61b904a2086439a003ecc01cce0db1 🚀
Parts:
- added C2: 10uf, Capacitor_SMD:CP_Elec_6.3x5.8, F.Cu at (102.5, 145.5)
- CON1: value SJ1-3523N -> 3.5mm jack
- Y1: value SG-8002CA -> 14.3181MHz
- moved C6 45.2 mm to (124.0, 155.5)
- moved C1 33.4 mm to (81.0, 142.5), turned to 0 degrees
- moved U2 13.1 mm to (134.5, 150.5)
- moved C19 12.4 mm to (114.0, 152.0)
- moved Y1 12.4 mm to (119.5, 150.5)
- moved C5 4.04 mm to (102.5, 156.0), turned to 180 degrees
- moved C15 3.04 mm to (133.0, 123.0)
- moved R8 3.03 mm to (140.5, 123.0)
- moved C16 2.85 mm to (133.0, 133.0)
- moved R9 2.76 mm to (140.5, 133.0)
- moved R1 2.31 mm to (73.0, 141.5)
- moved R2 2.31 mm to (73.0, 144.0)
- moved R3 2.31 mm to (73.0, 146.5)
- moved R4 2.31 mm to (73.0, 149.0)
- moved R5 2.31 mm to (73.0, 151.5)
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Routing:
- net /~{RESET}: track 11.0 -> 24.9 mm, vias 0 -> 2
- net /A1: track 27.6 -> 40.3 mm, vias 0 -> 2
- net /A0: track 23.8 -> 36.2 mm
- net /~{WR}: track 6.53 -> 18.6 mm
- net /DOAB: track 6.06 -> 16.9 mm
- net /~{RD}: track 6.69 -> 17.1 mm
- net /D0: track 7.22 -> 15.6 mm
- net /~{CS}: track 56.6 -> 63.5 mm, vias 0 -> 2
- net /D2: track 17.6 -> 24.2 mm
- net Net-(JP1-Pin_11): track 32.7 -> 26.8 mm
- net /D1: track 8.56 -> 14.1 mm
- net /DAC_CLK: track 8.23 -> 13.1 mm
- net /SMPAC: track 7.69 -> 11.9 mm
- net /D3: track 23.5 -> 26.9 mm
- net GND: track 31.6 -> 34.7 mm, vias 31 -> 25
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
Commit message: Deploying to main from @ electrified/rcbus-opl3@584da4a1b422c01a1dd6591974515cd0858dd859 🚀
Parts:
- moved C19 36.5 mm to (150.4, 149.0), turned to 0 degrees
- moved Y1 25.3 mm to (144.5, 146.5), turned to 90 degrees
- moved C6 11.5 mm to (123.5, 144.0)
- moved C7 7.58 mm to (118.3, 141.7)
- moved C9 7.12 mm to (127.1, 118.0), turned to 0 degrees
- moved C8 5.98 mm to (111.5, 127.8), turned to 180 degrees
- moved C10 5.95 mm to (123.2, 118.0), turned to 0 degrees
- moved U3 5.79 mm to (123.6, 135.8)
- moved U4 4.96 mm to (123.5, 123.0)
- moved C12 4.21 mm to (122.8, 128.7)
- moved R7 4.18 mm to (126.8, 128.7)
- moved C11 3.97 mm to (124.8, 128.7)
- moved C15 3.89 mm to (135.9, 120.4)
- moved C16 3.89 mm to (135.9, 130.4)
- moved R10 3.89 mm to (143.4, 124.4)
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Routing:
- net +5V: track 180.4 -> 242.3 mm
- net /D7: track 40.8 -> 16.0 mm
- net /D6: track 36.2 -> 13.7 mm
- net /D5: track 32.0 -> 11.4 mm
- net /D3: track 26.9 -> 8.45 mm
- net /D4: track 28.6 -> 10.3 mm
- net /DOAB: track 16.9 -> 34.4 mm
- net /D2: track 24.2 -> 7.18 mm
- net Net-(U3-MP): track 18.1 -> 8.56 mm
- net /~{CS}: track 63.5 -> 56.8 mm
- net Net-(U3-CV): track 25.1 -> 19.0 mm
- net Net-(U3-AOUT): track 11.8 -> 7.72 mm
- net /D1: track 14.1 -> 10.0 mm
- net /A1: track 40.3 -> 36.3 mm, vias 2 -> 1
- net Net-(CON1-PadT): track 14.7 -> 11.3 mm
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
Commit message: Deploying to main from @ electrified/rcbus-opl3@42ce7c760070e2171aef10dfe149ca65f88f18a5 🚀
Parts:
- moved C12 1.70 mm to (121.1, 128.7)
- moved C1 1.60 mm to (79.4, 142.4), turned to 180 degrees
- moved C11 0.90 mm to (123.9, 128.7)
- moved R7 0.85 mm to (125.9, 128.7)
- moved R11 0.39 mm to (143.4, 134.8)
- moved U1 0.27 mm to (86.3, 150.3)
- moved C15 0.19 mm to (135.9, 120.6)
- moved C16 0.19 mm to (135.9, 130.6)
- moved R10 0.19 mm to (143.4, 124.6)
- moved R8 0.19 mm to (143.4, 120.6)
- moved R9 0.19 mm to (143.4, 130.6)
Routing:
- net /DOAB: track 34.4 -> 21.5 mm, vias 0 -> 2
- net +5V: track 242.3 -> 233.1 mm
- net /~{CS}: track 56.8 -> 61.8 mm
- net Net-(JP1-Pin_7): track 28.5 -> 33.3 mm, vias 2 -> 0
- net /DAC_CLK: track 15.8 -> 19.8 mm
- net Net-(JP1-Pin_5): track 29.6 -> 33.3 mm
- net Net-(JP1-Pin_9): track 26.7 -> 29.8 mm
- net Net-(U3-MP): track 8.56 -> 11.4 mm
- net /~{IORQ}: track 54.2 -> 51.4 mm
- net GND: track 32.0 -> 29.5 mm, vias 22 -> 21
- net /A1: track 36.3 -> 38.3 mm
- net /A0: track 34.9 -> 36.8 mm
- net Net-(JP1-Pin_1): track 32.0 -> 30.3 mm, vias 0 -> 2
- net Net-(JP1-Pin_3): track 33.0 -> 31.5 mm
- net /D2: track 7.18 -> 8.32 mm
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- added copper zone on F.Cu, net +5V

Commit message: Deploying to main from @ electrified/rcbus-opl3@749e160d32f702c867f67f7984cd714a9df6dd66 🚀
Parts:
- moved C12 8.28 mm to (117.2, 121.4), turned to 90 degrees
Routing:
- net +5V: track 233.1 -> 229.1 mm
- net GND: track 29.5 -> 32.6 mm, vias 21 -> 23
- net Net-(U3-MP): track 11.4 -> 8.57 mm
- removed copper zone on F.Cu, net +5V

Commit message: Deploying to main from @ electrified/rcbus-opl3@bf3798d9d67c8703c79c41f51a896f3b0ec971bf 🚀
Parts:
- added REF**: Symbol_CreativeCommons_CopperTop_Type2_Big, Symbol:Symbol_CreativeCommons_CopperTop_Type2_Big, F.Cu at (53.0, 96.5)
- added REF**: Symbol_CC-Attribution_Silk_Small, electrified:Symbol_CC-Attribution_Silk_Small, B.Cu at (97.5, 159.0)
- added REF**: Symbol_CC-ShareAlike_Silk_Small, electrified:Symbol_CC-ShareAlike_Silk_Small, B.Cu at (91.5, 159.0)
- added REF**: Symbol_CreativeCommons_Silk_Type2_Small, electrified:Symbol_CreativeCommons_Silk_Type2_Small, B.Cu at (103.5, 159.0)
Routing:
- net /AUDIO_CH1: track 20.1 -> 20.8 mm
Other:
- board text added: "CC BY-SA https://creativecommons.org"

Commit message: Deploying to main from @ electrified/rcbus-opl3@76df5429c526e7a9126e9bdce83f90b253efb9f7 🚀
Parts:
- removed the REF** at (53.0, 96.5)
- C10: renamed from C2; value 10uf -> 10uF
- C3: renamed from C9; value 2.7nf -> 2.7nF
- C4: renamed from C10; value 2.7nf -> 2.7nF
- C5: renamed from C11; value 68pf -> 68pF
- C6: renamed from C16; value 10uf -> 10uF
- C7: renamed from C15; value 10uf -> 10uF
- renumbered C8 to C1, C6 to C11, C7 to C12, C19 to C13, C12 to C2, C1 to C8, C5 to C9, R7 to R1, R3 to R10, R6 to R11, R8 to R2, R9 to R3, R10 to R4, R11 to R5, R5 to R6, R4 to R7, R2 to R8, R1 to R9, U3 to U1, U4 to U2, U1 to U3, U2 to U4
Routing:
- net GND: vias 23 -> 86

Commit message: Deploying to main from @ electrified/rcbus-opl3@4d18163650932ad5441b7bd8b3289f36741a7241 🚀
Parts:
- renumbered C6 to C2, C4 to C3, C3 to C4, C2 to C5, C5 to C6, REF** to G3, REF** to G4, REF** to G5, R4 to R2, R2 to R3, R3 to R4, R7 to R6, R6 to R7, U2 to U1, U1 to U2
